Commit message: stl, dae 파일 읽는 경로 수정

File: urdf/_d435.urdf.xacro (robot description, xacro)
@@ -53,5 +53,5 @@
         <geometry>
           <!-- <box size="${d435_cam_width} ${d435_cam_height} ${d435_cam_depth}"/> -->
-	        <mesh filename="package://rdv_3d_mapping_camera/meshes/d435.dae" />
+	        <mesh filename="package://ros_rdv_3d_mapping_camera_model/meshes/d435.dae" />
         </geometry>
       </visual>

File: urdf/_usb_plug.urdf.xacro (robot description, xacro)
@@ -20,5 +20,5 @@
         <geometry>
           <!--box size="0.044850 0.008 0.0185" /-->
-          <mesh filename="package://rdv_3d_mapping_camera/meshes/plug.stl" />
+          <mesh filename="package://ros_rdv_3d_mapping_camera_model/meshes/plug.stl" />
         </geometry>
         <material name="plastic"/>
@@ -28,5 +28,5 @@
         <geometry>
           <!--box size="0.044850 0.008 0.0185" /-->
-          <mesh filename="package://rdv_3d_mapping_camera/meshes/plug_collision.stl" />
+          <mesh filename="package://ros_rdv_3d_mapping_camera_model/meshes/plug_collision.stl" />
         </geometry>
       </collision>
