Commit message: stl 모델의 scale과 offset 문제 해결.

File: urdf/rdv_3d_mapping_camera.urdf.xacro (robot description, xacro)
@@ -43,15 +43,19 @@
     <link name="top_link" parent="top_pole_joint" >
         <visual>
+            <origin rpy="0 0 0" xyz="0 0 0"/>
             <geometry>
+                <!-- <mesh filename="package://rdv_3d_mapping_camera/meshes/ASSY_BEER_RANGE_360_angle.stl" scale=".0254 .0254 .0254"/> -->
                 <mesh filename="package://rdv_3d_mapping_camera/meshes/ASSY_BEER_RANGE_360_angle.stl" />
             </geometry>
-            <origin rpy="0 0 0" xyz="0 0 0.1"/>
-            <material name="green">
-                <color rgba="0 1 0 1"/>
-            </material>
         </visual>
     </link>
-  <xacro:sensor_d435 parent="top_link" use_nominal_extrinsics="$(arg use_nominal_extrinsics)">
-    <origin xyz="0 0 0.5" rpy="1.57 0 0"/>
+<!--
+  <link name="top_link" parent="top_pole_joint" />
+-->
+  <xacro:sensor_d435 parent="top_link" name="camera_01"  use_nominal_extrinsics="$(arg use_nominal_extrinsics)">
+    <origin xyz="0.1 0 0" rpy="1.57 0 0"/>
+  </xacro:sensor_d435>
+  <xacro:sensor_d435 parent="top_link" name="camera_02"  use_nominal_extrinsics="$(arg use_nominal_extrinsics)">
+    <origin xyz="-0.1 0 0" rpy="1.57 0 3.1456"/>
   </xacro:sensor_d435>
 </robot>

Commit message: 10대의 카메라가 위치할 TF생성, 카메라 위치 Pose를 자동으로 계산하는 C++ 코드 추가.

File: urdf/rdv_3d_mapping_camera.urdf.xacro (robot description, xacro)
@@ -43,5 +43,5 @@
     <link name="top_link" parent="top_pole_joint" >
         <visual>
-            <origin rpy="0 0 0" xyz="0 0 0"/>
+            <origin rpy="0 0 1.570796" xyz="0 0 0"/>
             <geometry>
                 <!-- <mesh filename="package://rdv_3d_mapping_camera/meshes/ASSY_BEER_RANGE_360_angle.stl" scale=".0254 .0254 .0254"/> -->
@@ -51,11 +51,128 @@
     </link>
 <!--
-  <link name="top_link" parent="top_pole_joint" />
+    <joint name="camera_01_joint" type="fixed">
+      <parent link="top_link"/>
+      <child link="camera_01_pose_link"/>
+      <origin xyz="0.06855 0 0.04930" rpy="1.57 0.5235986666666667 0"/>
+    </joint>
+    <link name="camera_01_pose_link" />
+    <joint name="camera_02_joint" type="fixed">
+      <parent link="top_link"/>
+      <child link="camera_02_pose_link"/>
+      <origin xyz="0.06855 0 0.04930" rpy="1.57 0.5235986666666667 0"/>
+    </joint>
+    <link name="camera_02_pose_link" />
 -->
+    <joint name="camera_00_joint" type="fixed">
+    <parent link="top_link"/>
+    <child link="camera_00_pose_link"/>
+    <origin xyz="0.068550 0.000000 0.04930" rpy="1.57 0.5235986666666667 0.000000"/>
+</joint>
+<link name="camera_00_pose_link" />
+<joint name="camera_01_joint" type="fixed">
+    <parent link="top_link"/>
+    <child link="camera_01_pose_link"/>
+    <origin xyz="0.055458 0.040293 0.04930" rpy="1.57 0.5235986666666667 0.628318"/>
+</joint>
+<link name="camera_01_pose_link" />
+<joint name="camera_02_joint" type="fixed">
+    <parent link="top_link"/>
+    <child link="camera_02_pose_link"/>
+    <origin xyz="0.021183 0.065195 0.04930" rpy="1.57 0.5235986666666667 1.256637"/>
+</joint>
+<link name="camera_02_pose_link" />
+<joint name="camera_03_joint" type="fixed">
+    <parent link="top_link"/>
+    <child link="camera_03_pose_link"/>
+    <origin xyz="-0.021183 0.065195 0.04930" rpy="1.57 0.5235986666666667 1.884955"/>
+</joint>
+<link name="camera_03_pose_link" />
+<joint name="camera_04_joint" type="fixed">
+    <parent link="top_link"/>
+    <child link="camera_04_pose_link"/>
+    <origin xyz="-0.055458 0.040293 0.04930" rpy="1.57 0.5235986666666667 2.513274"/>
+</joint>
+<link name="camera_04_pose_link" />
+<joint name="camera_05_joint" type="fixed">
+    <parent link="top_link"/>
+    <child link="camera_05_pose_link"/>
+    <origin xyz="-0.068550 0.000000 0.04930" rpy="1.57 0.5235986666666667 3.141592"/>
+</joint>
+<link name="camera_05_pose_link" />
+<joint name="camera_06_joint" type="fixed">
+    <parent link="top_link"/>
+    <child link="camera_06_pose_link"/>
+    <origin xyz="-0.055458 -0.040293 0.04930" rpy="1.57 0.5235986666666667 3.769910"/>
+</joint>
+<link name="camera_06_pose_link" />
+<joint name="camera_07_joint" type="fixed">
+    <parent link="top_link"/>
+    <child link="camera_07_pose_link"/>
+    <origin xyz="-0.021183 -0.065195 0.04930" rpy="1.57 0.5235986666666667 4.398229"/>
+</joint>
+<link name="camera_07_pose_link" />
+<joint name="camera_08_joint" type="fixed">
+    <parent link="top_link"/>
+    <child link="camera_08_pose_link"/>
+    <origin xyz="0.021183 -0.065195 0.04930" rpy="1.57 0.5235986666666667 5.026547"/>
+</joint>
+<link name="camera_08_pose_link" />
+<joint name="camera_09_joint" type="fixed">
+    <parent link="top_link"/>
+    <child link="camera_09_pose_link"/>
+    <origin xyz="0.055458 -0.040293 0.04930" rpy="1.57 0.5235986666666667 5.654866"/>
+</joint>
+<link name="camera_09_pose_link" />
+<!--
+    <joint name="camera_03_joint" type="fixed">
+      <parent link="top_link"/>
+      <child link="camera_03_pose_link"/>
+      <origin xyz="${(cos_degree_36*3) * camera_r} ${(sin_degree_36*3) * camera_r} 0.04930" rpy="1.57 0.5235986666666667 ${radian_36_degree*3}"/>
+    </joint>
+    <link name="camera_03_pose_link" />
+    <joint name="camera_04_joint" type="fixed">
+      <parent link="top_link"/>
+      <child link="camera_04_pose_link"/>
+      <origin xyz="${(cos_degree_36*4) * camera_r} ${(sin_degree_36*4) * camera_r} 0.04930" rpy="1.57 0.5235986666666667 ${radian_36_degree*4}"/>
+    </joint>
+    <link name="camera_04_pose_link" />
+    <joint name="camera_05_joint" type="fixed">
+      <parent link="top_link"/>
+      <child link="camera_05_pose_link"/>
+      <origin xyz="${(cos_degree_36*5) * camera_r} ${(sin_degree_36*5) * camera_r} 0.04930" rpy="1.57 0.5235986666666667 ${radian_36_degree*5}"/>
+    </joint>
+    <link name="camera_05_pose_link" />
+    <joint name="camera_06_joint" type="fixed">
+      <parent link="top_link"/>
+      <child link="camera_06_pose_link"/>
+      <origin xyz="${(cos_degree_36*6) * camera_r} ${(sin_degree_36*6) * camera_r} 0.04930" rpy="1.57 0.5235986666666667 ${radian_36_degree*6}"/>
+    </joint>
+    <link name="camera_06_pose_link" />
+    <joint name="camera_07_joint" type="fixed">
+      <parent link="top_link"/>
+      <child link="camera_07_pose_link"/>
+      <origin xyz="${(cos_degree_36*7) * camera_r} ${(sin_degree_36*7) * camera_r} 0.04930" rpy="1.57 0.5235986666666667 ${radian_36_degree*7}"/>
+    </joint>
+    <link name="camera_07_pose_link" />
+    <joint name="camera_08_joint" type="fixed">
+      <parent link="top_link"/>
+      <child link="camera_08_pose_link"/>
+      <origin xyz="${(cos_degree_36*8) * camera_r} ${(sin_degree_36*8) * camera_r} 0.04930" rpy="1.57 0.5235986666666667 ${radian_36_degree*8}"/>
+    </joint>
+    <link name="camera_08_pose_link" />
+    <joint name="camera_09_joint" type="fixed">
+      <parent link="top_link"/>
+      <child link="camera_09_pose_link"/>
+      <origin xyz="${(cos_degree_36*9) * camera_r} ${(sin_degree_36*9) * camera_r} 0.04930" rpy="1.57 0.5235986666666667 ${radian_36_degree*9}"/>
+    </joint>
+    <link name="camera_09_pose_link" />
+-->
+<!--
   <xacro:sensor_d435 parent="top_link" name="camera_01"  use_nominal_extrinsics="$(arg use_nominal_extrinsics)">
-    <origin xyz="0.1 0 0" rpy="1.57 0 0"/>
+    <origin xyz="0.07834 0.0125 0.04596" rpy="1.57 0.5235986666666667 0"/>
   </xacro:sensor_d435>
   <xacro:sensor_d435 parent="top_link" name="camera_02"  use_nominal_extrinsics="$(arg use_nominal_extrinsics)">
     <origin xyz="-0.1 0 0" rpy="1.57 0 3.1456"/>
   </xacro:sensor_d435>
+-->
 </robot>

Commit message: 10대의 카메라를 TF(Joint)를 기준으로 위치 시킴.

File: urdf/rdv_3d_mapping_camera.urdf.xacro (robot description, xacro)
@@ -3,4 +3,5 @@
   <xacro:arg name="use_nominal_extrinsics" default="false"/>
   <xacro:include filename="$(find rdv_3d_mapping_camera)/urdf/_d435.urdf.xacro" />
+  <xacro:include filename="$(find rdv_3d_mapping_camera)/urdf/_3d_mapping_camera_frame.urdf.xacro" />
 <!--
   <link name="base_link" />
@@ -36,142 +37,13 @@
       </visual>
   </link>
-  <joint name="top_pole_joint" type="fixed">
-      <parent link="pole_link"/>
-      <child link="top_link"/>
-      <origin xyz="0.0 0.0 2.0" rpy="0 0 0"/>
-  </joint>
-    <link name="top_link" parent="top_pole_joint" >
-        <visual>
-            <origin rpy="0 0 1.570796" xyz="0 0 0"/>
-            <geometry>
-                <!-- <mesh filename="package://rdv_3d_mapping_camera/meshes/ASSY_BEER_RANGE_360_angle.stl" scale=".0254 .0254 .0254"/> -->
-                <mesh filename="package://rdv_3d_mapping_camera/meshes/ASSY_BEER_RANGE_360_angle.stl" />
-            </geometry>
-        </visual>
-    </link>
+    <xacro:camera_frame parent="pole_link" name="camera_frame">
+    <origin xyz="0 0 0" rpy="0 0 0"/>
+  </xacro:camera_frame>
 <!--
-    <joint name="camera_01_joint" type="fixed">
-      <parent link="top_link"/>
-      <child link="camera_01_pose_link"/>
-      <origin xyz="0.06855 0 0.04930" rpy="1.57 0.5235986666666667 0"/>
-    </joint>
-    <link name="camera_01_pose_link" />
-    <joint name="camera_02_joint" type="fixed">
-      <parent link="top_link"/>
-      <child link="camera_02_pose_link"/>
-      <origin xyz="0.06855 0 0.04930" rpy="1.57 0.5235986666666667 0"/>
-    </joint>
-    <link name="camera_02_pose_link" />
--->
-    <joint name="camera_00_joint" type="fixed">
-    <parent link="top_link"/>
-    <child link="camera_00_pose_link"/>
-    <origin xyz="0.068550 0.000000 0.04930" rpy="1.57 0.5235986666666667 0.000000"/>
-</joint>
-<link name="camera_00_pose_link" />
-<joint name="camera_01_joint" type="fixed">
-    <parent link="top_link"/>
-    <child link="camera_01_pose_link"/>
-    <origin xyz="0.055458 0.040293 0.04930" rpy="1.57 0.5235986666666667 0.628318"/>
-</joint>
-<link name="camera_01_pose_link" />
-<joint name="camera_02_joint" type="fixed">
-    <parent link="top_link"/>
-    <child link="camera_02_pose_link"/>
-    <origin xyz="0.021183 0.065195 0.04930" rpy="1.57 0.5235986666666667 1.256637"/>
-</joint>
-<link name="camera_02_pose_link" />
-<joint name="camera_03_joint" type="fixed">
-    <parent link="top_link"/>
-    <child link="camera_03_pose_link"/>
-    <origin xyz="-0.021183 0.065195 0.04930" rpy="1.57 0.5235986666666667 1.884955"/>
-</joint>
-<link name="camera_03_pose_link" />
-<joint name="camera_04_joint" type="fixed">
-    <parent link="top_link"/>
-    <child link="camera_04_pose_link"/>
-    <origin xyz="-0.055458 0.040293 0.04930" rpy="1.57 0.5235986666666667 2.513274"/>
-</joint>
-<link name="camera_04_pose_link" />
-<joint name="camera_05_joint" type="fixed">
-    <parent link="top_link"/>
-    <child link="camera_05_pose_link"/>
-    <origin xyz="-0.068550 0.000000 0.04930" rpy="1.57 0.5235986666666667 3.141592"/>
-</joint>
-<link name="camera_05_pose_link" />
-<joint name="camera_06_joint" type="fixed">
-    <parent link="top_link"/>
-    <child link="camera_06_pose_link"/>
-    <origin xyz="-0.055458 -0.040293 0.04930" rpy="1.57 0.5235986666666667 3.769910"/>
-</joint>
-<link name="camera_06_pose_link" />
-<joint name="camera_07_joint" type="fixed">
-    <parent link="top_link"/>
-    <child link="camera_07_pose_link"/>
-    <origin xyz="-0.021183 -0.065195 0.04930" rpy="1.57 0.5235986666666667 4.398229"/>
-</joint>
-<link name="camera_07_pose_link" />
-<joint name="camera_08_joint" type="fixed">
-    <parent link="top_link"/>
-    <child link="camera_08_pose_link"/>
-    <origin xyz="0.021183 -0.065195 0.04930" rpy="1.57 0.5235986666666667 5.026547"/>
-</joint>
-<link name="camera_08_pose_link" />
-<joint name="camera_09_joint" type="fixed">
-    <parent link="top_link"/>
-    <child link="camera_09_pose_link"/>
-    <origin xyz="0.055458 -0.040293 0.04930" rpy="1.57 0.5235986666666667 5.654866"/>
-</joint>
-<link name="camera_09_pose_link" />
-<!--
-    <joint name="camera_03_joint" type="fixed">
-      <parent link="top_link"/>
-      <child link="camera_03_pose_link"/>
-      <origin xyz="${(cos_degree_36*3) * camera_r} ${(sin_degree_36*3) * camera_r} 0.04930" rpy="1.57 0.5235986666666667 ${radian_36_degree*3}"/>
-    </joint>
-    <link name="camera_03_pose_link" />
-    <joint name="camera_04_joint" type="fixed">
-      <parent link="top_link"/>
-      <child link="camera_04_pose_link"/>
-      <origin xyz="${(cos_degree_36*4) * camera_r} ${(sin_degree_36*4) * camera_r} 0.04930" rpy="1.57 0.5235986666666667 ${radian_36_degree*4}"/>
-    </joint>
-    <link name="camera_04_pose_link" />
-    <joint name="camera_05_joint" type="fixed">
-      <parent link="top_link"/>
-      <child link="camera_05_pose_link"/>
-      <origin xyz="${(cos_degree_36*5) * camera_r} ${(sin_degree_36*5) * camera_r} 0.04930" rpy="1.57 0.5235986666666667 ${radian_36_degree*5}"/>
-    </joint>
-    <link name="camera_05_pose_link" />
-    <joint name="camera_06_joint" type="fixed">
-      <parent link="top_link"/>
-      <child link="camera_06_pose_link"/>
-      <origin xyz="${(cos_degree_36*6) * camera_r} ${(sin_degree_36*6) * camera_r} 0.04930" rpy="1.57 0.5235986666666667 ${radian_36_degree*6}"/>
-    </joint>
-    <link name="camera_06_pose_link" />
-    <joint name="camera_07_joint" type="fixed">
-      <parent link="top_link"/>
-      <child link="camera_07_pose_link"/>
-      <origin xyz="${(cos_degree_36*7) * camera_r} ${(sin_degree_36*7) * camera_r} 0.04930" rpy="1.57 0.5235986666666667 ${radian_36_degree*7}"/>
-    </joint>
-    <link name="camera_07_pose_link" />
-    <joint name="camera_08_joint" type="fixed">
-      <parent link="top_link"/>
-      <child link="camera_08_pose_link"/>
-      <origin xyz="${(cos_degree_36*8) * camera_r} ${(sin_degree_36*8) * camera_r} 0.04930" rpy="1.57 0.5235986666666667 ${radian_36_degree*8}"/>
-    </joint>
-    <link name="camera_08_pose_link" />
-    <joint name="camera_09_joint" type="fixed">
-      <parent link="top_link"/>
-      <child link="camera_09_pose_link"/>
-      <origin xyz="${(cos_degree_36*9) * camera_r} ${(sin_degree_36*9) * camera_r} 0.04930" rpy="1.57 0.5235986666666667 ${radian_36_degree*9}"/>
-    </joint>
-    <link name="camera_09_pose_link" />
--->
-<!--
-  <xacro:sensor_d435 parent="top_link" name="camera_01"  use_nominal_extrinsics="$(arg use_nominal_extrinsics)">
-    <origin xyz="0.07834 0.0125 0.04596" rpy="1.57 0.5235986666666667 0"/>
+  <xacro:sensor_d435 parent="camera_00_pose_link" name="camera_01"  use_nominal_extrinsics="$(arg use_nominal_extrinsics)">
+    <origin xyz="0 0 0" rpy="0 0 0"/>
   </xacro:sensor_d435>
-  <xacro:sensor_d435 parent="top_link" name="camera_02"  use_nominal_extrinsics="$(arg use_nominal_extrinsics)">
-    <origin xyz="-0.1 0 0" rpy="1.57 0 3.1456"/>
+  <xacro:sensor_d435 parent="camera_01_pose_link" name="camera_02"  use_nominal_extrinsics="$(arg use_nominal_extrinsics)">
+    <origin xyz="0 0 0" rpy="0 0 0"/>
   </xacro:sensor_d435>
 -->

Commit message: 카메라의 폴대를 회색으로 변경

File: urdf/rdv_3d_mapping_camera.urdf.xacro (robot description, xacro)
@@ -14,6 +14,6 @@
           </geometry>
           <origin rpy="0 0 0" xyz="0 0 0.005"/>
-          <material name="yellow">
-              <color rgba="1 1 0 1"/>
+          <material name="">
+              <color rgba="0.5 0.5 0.5 1"/>
           </material>
       </visual>
@@ -30,6 +30,6 @@
           </geometry>
           <origin rpy="0 0 0" xyz="0 0 0.75"/>
-          <material name="red">
-              <color rgba="1 0 0 1"/>
+          <material name="">
+              <color rgba="0.5 0.5 0.5 1"/>
           </material>
       </visual>
